Commit message: Normal commit

File: ros2_control_demos/example_2/description/urdf/diffbot.urdf.xacro (robot description, xacro)
@@ -1,15 +1,18 @@
 <?xml version="1.0"?>
-<!-- Basic differential drive mobile base -->
+<!-- Basic differential drive mobile base with 4 wheels -->
 <robot xmlns:xacro="http://www.ros.org/wiki/xacro" name="diffdrive_robot">
   <xacro:arg name="prefix" default="" />
   <xacro:arg name="use_mock_hardware" default="false" />
   <xacro:arg name="use_sim_time" default="false" />
-  <xacro:include filename="$(find ros2_control_demo_description)/diffbot/urdf/diffbot_description.urdf.xacro" />
+  <xacro:include filename="$(find ros2_control_demo_description)/diffbot/urdf/diffbot_description_4wheels.urdf.xacro" />
   <!-- Import Rviz colors -->
   <xacro:include filename="$(find ros2_control_demo_description)/diffbot/urdf/diffbot.materials.xacro" />
   <!-- Import diffbot ros2_control description -->
-  <xacro:include filename="$(find ros2_control_demo_example_2)/ros2_control/diffbot.ros2_control.xacro" />
-  <xacro:diffbot prefix="$(arg prefix)" />
+  <xacro:include filename="$(find ros2_control_demo_example_2)/ros2_control/diffbot_4wheels.ros2_control.xacro" />
+  <xacro:diffbot_4wheels prefix="$(arg prefix)" />
   <xacro:diffbot_ros2_control
-    name="DiffBot" prefix="$(arg prefix)" use_mock_hardware="$(arg use_mock_hardware)" use_sim_time="$(arg use_sim_time)"/>
+    name="DiffBot"
+    prefix="$(arg prefix)"
+    use_mock_hardware="$(arg use_mock_hardware)"
+    use_sim_time="$(arg use_sim_time)"/>
 </robot>

File: ros2_control_demos/ros2_control_demo_description/diffbot/urdf/diffbot_description_4wheels.urdf.xacro (robot description, xacro)
@@ -1,10 +1,10 @@
 <?xml version="1.0"?>
 <robot xmlns:xacro="http://www.ros.org/wiki/xacro">
-  <xacro:macro name="diffbot" params="prefix">
+  <xacro:macro name="diffbot_4wheels" params="prefix">
   <!-- Constants for robot dimensions -->
   <xacro:property name="PI" value="3.1415926535897931"/>
   <xacro:property name="base_mass" value="0.3" /> <!-- arbitrary value for base mass -->
   <xacro:property name="base_width" value="0.1" />
-  <xacro:property name="base_length" value="0.3" /> <!-- Increased length to accommodate 4 wheels -->
+  <xacro:property name="base_length" value="0.3" /> <!-- Increased length for 4-wheeled model -->
   <xacro:property name="base_height" value="0.05" />
   <xacro:property name="wheel_mass" value="0.3" /> <!-- arbitrary value for wheel mass -->
@@ -12,6 +12,4 @@
   <xacro:property name="wheel_radius" value="0.015" />
   <xacro:property name="wheel_separation_x" value="0.2" /> <!-- Separation between front and rear wheels -->
-  <xacro:property name="caster_wheel_mass" value="0.1" /> <!-- arbitrary value for caster wheel mass -->
-  <xacro:property name="caster_wheel_radius" value="0.015" />
   <xacro:property name="z_offset" value="-${base_height/2}" /> <!-- Space btw top of beam and the each joint -->
   <!-- Base Link -->
@@ -39,5 +37,5 @@
       </inertial>
     </link>
-    <!-- Front left wheel -->
+    <!-- Front Left Wheel -->
     <joint name="${prefix}front_left_wheel_joint" type="continuous">
       <parent link="${prefix}base_link"/>
@@ -71,9 +69,9 @@
         </inertial>
       </link>
-    <!-- Rear left wheel -->
+    <!-- Rear Left Wheel -->
     <joint name="${prefix}rear_left_wheel_joint" type="continuous">
       <parent link="${prefix}base_link"/>
       <child link="${prefix}rear_left_wheel"/>
-      <origin xyz="${-wheel_separation_x/2} -${base_width/2} ${z_offset}" rpy="0 0 0"/>
+      <origin xyz="-${wheel_separation_x/2} -${base_width/2} ${z_offset}" rpy="0 0 0"/>
       <axis xyz="0 1 0"/>
       <dynamics damping="0.2"/>
@@ -103,5 +101,5 @@
         </inertial>
       </link>
-    <!-- Front right wheel -->
+    <!-- Front Right Wheel -->
     <joint name="${prefix}front_right_wheel_joint" type="continuous">
       <parent link="${prefix}base_link"/>
@@ -135,9 +133,9 @@
         </inertial>
       </link>
-    <!-- Rear right wheel -->
+    <!-- Rear Right Wheel -->
     <joint name="${prefix}rear_right_wheel_joint" type="continuous">
       <parent link="${prefix}base_link"/>
       <child link="${prefix}rear_right_wheel"/>
-      <origin xyz="${-wheel_separation_x/2} ${base_width/2} ${z_offset}" rpy="0 0 0"/>
+      <origin xyz="-${wheel_separation_x/2} ${base_width/2} ${z_offset}" rpy="0 0 0"/>
       <axis xyz="0 1 0"/>
       <dynamics damping="0.2"/>

File: submodules/ros_odrive/odrive_botwheel_explorer/description/urdf/diffbot.ros2_control.xacro (robot description, xacro)
@@ -15,9 +15,17 @@
         </hardware>
       </xacro:if>
-      <joint name="${prefix}left_wheel_joint">
+      <!-- Left side wheels with their respective ODrive node IDs -->
+      <joint name="${prefix}front_left_wheel_joint">
         <param name="node_id">0</param>
       </joint>
-      <joint name="${prefix}right_wheel_joint">
+      <joint name="${prefix}rear_left_wheel_joint">
         <param name="node_id">1</param>
+      </joint>
+      <!-- Right side wheels with their respective ODrive node IDs -->
+      <joint name="${prefix}front_right_wheel_joint">
+        <param name="node_id">2</param>
+      </joint>
+      <joint name="${prefix}rear_right_wheel_joint">
+        <param name="node_id">3</param>
       </joint>
     </ros2_control>
